File: HW2/Schematic.brd (EAGLE design)
At the start: 100 x 80 mm, 21 parts, among them J1 USBSMD

Commit message: board complete!
Parts:
- removed C4, C5, C6, C7: 0.1uF, pic32_library:E2,5-5
- removed J2: (no value), pic32_library:1X05
- moved J5 99.6 mm to (44.5, 20.3), turned to 90 degrees
- moved C1 81.9 mm to (40.6, 44.5)
- moved R2 77.5 mm to (30.5, 47.0), turned to 180 degrees
- moved J4 65.4 mm to (8.89, 22.9), turned to 90 degrees
- moved U$5 64.1 mm to (33.0, 3.81)
- moved U$3 63.6 mm to (17.8, 19.1), turned to 90 degrees
- moved J1 63.5 mm to (44.5, 6.35), turned to 180 degrees
- moved U$2 63.1 mm to (22.9, 5.08), turned to 180 degrees
- moved U$1 61.9 mm to (26.7, 26.7), turned to 270 degrees
- moved U$4 59.2 mm to (3.81, 3.81), turned to 180 degrees
- moved LED1 57.1 mm to (10.2, 3.81), turned to 180 degrees
- moved R1 51.1 mm to (15.2, 33.0), turned to 90 degrees
- moved J3 50.3 mm to (15.2, 48.3), turned to 180 degrees
- moved C2 40.9 mm to (16.5, 10.2), turned to 180 degrees
- moved C3 37.4 mm to (5.08, 16.5)
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Connections:
- net +3V3: now also R2.1; no longer C4.+, C5.+, C6.+, C7.-
- net GND: no longer C4.-, C5.-, C6.-, C7.+
- net USBID: now also J1.ID
Routing:
- net +3V3: track 0.00 -> 124.5 mm, vias 0 -> 3
- net +5V: track 0.00 -> 56.4 mm, vias 0 -> 2
- net B4: track 0.00 -> 54.0 mm, vias 0 -> 1
- net A4: track 0.00 -> 47.2 mm
- net N$3: track 0.00 -> 39.1 mm, vias 0 -> 3
- net N$2: track 0.00 -> 30.8 mm
- net N$1: track 0.00 -> 29.0 mm, vias 0 -> 1
- net MCLR: track 0.00 -> 27.8 mm
- net PGEC1: track 0.00 -> 26.8 mm
- net B7: track 0.00 -> 23.4 mm, vias 0 -> 1
- net PGED1: track 0.00 -> 23.3 mm
- net B8: track 0.00 -> 22.6 mm, vias 0 -> 1
- net B9: track 0.00 -> 21.1 mm, vias 0 -> 1
- net USBID: track 0.00 -> 19.9 mm, vias 0 -> 1
- net GND: track 0.00 -> 17.8 mm
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- added copper zone on layer 16, net GND
Other:
- board size 100 x 80 mm -> 50 x 50 mm

Commit message: gerber files complete! PCB ready for printing
Parts:
- removed J1: USBSMD, pic32_library:USB-MINIB
- added J2: USB-MB-H, pic32_library:USB-MB-H
- moved J4 9.92 mm to (1.27, 16.5)
- moved J5 5.85 mm to (48.9, 16.5)
- moved C3 5.08 mm to (5.08, 11.4)
- moved C1 3.81 mm to (40.6, 40.6)
- turned U$4 to 270 degrees
- renumbered U$1 to PIC32
Connections:
- net GND: now also J2.GND; no longer J1.GND
- net N$2: now also J2.D-; no longer J1.D-
- net N$3: now also J2.D+; no longer J1.D+
- net N$6: now also J2.VBUS; no longer J1.VBUS
- net USBID: now also J2.ID; no longer J1.ID
Routing:
- net GND: track 17.8 -> 0.00 mm
- net B3: track 17.6 -> 27.5 mm
- net A1: track 16.1 -> 26.0 mm
- net A0: track 16.1 -> 26.0 mm
- net B4: track 54.0 -> 63.9 mm, vias 1 -> 2
- net B2: track 17.6 -> 26.7 mm
- net USBID: track 19.9 -> 24.8 mm, vias 1 -> 0
- net B15: track 14.0 -> 18.8 mm
- net B14: track 14.0 -> 18.8 mm
- net B13: track 14.0 -> 18.8 mm
- net N$2: track 30.8 -> 35.5 mm, vias 0 -> 1
- net A4: track 47.2 -> 42.9 mm
- net N$1: track 29.0 -> 25.2 mm
- net +5V: track 56.4 -> 54.0 mm
- net N$6: track 10.9 -> 12.7 mm
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Other:
- board text added: "3.3V"
- board text added: "5V"
- board text added: ">"
- board text added: "A0"
- board text added: "A1"
- board text added: "A4"
- board text added: "B13"
- board text added: "B14"
- board text added: "B15"
- board text added: "B2"
- board text added: "B3"
- board text added: "B4"
- board text added: "B7"
- board text added: "B8"
- board text added: "B9"
- board text added: "GND"
- board text added: "I"
- board text added: "Karl zur Loye"
- board text added: "RESET"
- board text added: "USER"
