File: HW2/Schematic.sch (EAGLE design)
At the start: 3 parts

Commit message: schematic done
Parts:
- added C1: 10uF, pic32_library:CPOL-USE2.5-5
- added C2, C3, C4, C5, C6, C7: 0.1uF, pic32_library:CPOL-USE2.5-5
- added J1: USBSMD, pic32_library:USBSMD
- added J2: (no value), pic32_library:M05PTH
- added J3: (no value), pic32_library:M06SILK_FEMALE_PTH
- added J4, J5: (no value), pic32_library:M08SILK_FEMALE_PTH
- added R2: 10K, pic32_library:R-US_0207/10
- added U$2: MCP1702, pic32_library:MCP1702
- added U$3: RESONATOR, pic32_library:RESONATOR
- added U$4, U$6: PUSH_BUTTON, pic32_library:PUSH_BUTTON
- added U$5: SLIDE-SWITCH, pic32_library:SLIDE-SWITCH
- R1: value (none) -> 10K
Connections:
- new net +5V: C2.+, J5.2, U$1.15.5V, U$2.2.VIN, U$5.3.R
- new net A0: J4.8, U$1.2.
- new net A1: J4.7, U$1.3.
- new net A4: J4.3, LED1.A, U$1.12.RA4
- new net B13: J5.6, U$1.24.
- new net B14: J5.7, U$1.25.
- new net B15: J5.8, U$1.26.
- new net B2: J4.6, U$1.6.
- new net B3: J4.5, U$1.7.
- new net B4: J4.4, R1.2, U$1.11.RB4, U$4.2.R
- new net B7: J5.3, U$1.16.
- new net B8: J5.4, U$1.17.
- new net B9: J5.5, U$1.18.
- new net MCLR: J3.1, R2.2, U$1.1.MCLR, U$6.1.L
- new net N$1: C1.+, U$1.20.10UF
- new net N$2: J1.D-, U$1.22.D-
- new net N$3: J1.D+, U$1.21.D+
- new net N$4: U$1.9.OSC1, U$3.3.R
- new net N$5: U$1.10.OSC2, U$3.1.L
- new net N$6: J1.VBUS, U$5.1.5V
- new net N$9: J3.6
- new net PGEC1: J3.5, U$1.5.PGEC1
- new net PGED1: J3.4, U$1.4.PGED1
- new net USBID: U$1.14.USBID
- net +3V3: now also C3.+, C4.+, C5.+, C6.+, C7.-, J3.2, J4.2, R1.1, U$1.13.GND, U$2.3.VOUT; no longer U$1.8.3.3V
- net GND: now also C1.-, C2.-, C3.-, C4.-, C5.-, C6.-, C7.+, J1.GND, J3.3, J4.1, J5.1, LED1.C, U$1.8.3.3V, U$2.1.GND, U$3.2.GND, U$4.1.L, U$6.2.R; no longer U$1.13.GND
Other:
- moved on the sheet: LED1, R1

Commit message: board complete!
Parts:
- removed C4, C5, C6, C7: 0.1uF, pic32_library:CPOL-USE2.5-5
- removed J2: (no value), pic32_library:M05PTH
Connections:
- net +3V3: now also R2.1; no longer C4.+, C5.+, C6.+, C7.-
- net GND: now also J1.1.GND; no longer C4.-, C5.-, C6.-, C7.+, J1.GND
- net N$2: now also J1.4.D-; no longer J1.D-
- net N$3: now also J1.3.D+; no longer J1.D+
- net N$6: now also J1.5.VBUS; no longer J1.VBUS
- net USBID: now also J1.2.ID
Changed lines of the file:
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@@
 <part name="GND8" library="pic32_library" deviceset="GND" device=""/>
 <part name="+3V5" library="pic32_library" deviceset="+3V3" device=""/>
-<part name="C4" library="pic32_library" deviceset="CPOL-US" device="E2.5-5" value="0.1uF"/>
-<part name="C5" library="pic32_library" deviceset="CPOL-US" device="E2.5-5" value="0.1uF"/>
-<part name="C6" library="pic32_library" deviceset="CPOL-US" device="E2.5-5" value="0.1uF"/>
-<part name="+3V6" library="pic32_library" deviceset="+3V3" device=""/>
-<part name="J2" library="pic32_library" deviceset="M05" device="PTH"/>
-<part name="+3V7" library="pic32_library" deviceset="+3V3" device=""/>
 <part name="U$4" library="pic32_library" deviceset="PUSH_BUTTON" device=""/>
 <part name="GND9" library="pic32_library" deviceset="GND" device=""/>
-<part name="C7" library="pic32_library" deviceset="CPOL-US" device="E2.5-5" value="0.1uF"/>
 <part name="GND10" library="pic32_library" deviceset="GND" device=""/>
 <part name="+3V3" library="pic32_library" deviceset="+3V3" device=""/>
@@
 <instance part="GND8" gate="1" x="137.16" y="50.8" rot="R90"/>
 <instance part="+3V5" gate="G$1" x="119.38" y="50.8" rot="R90"/>
-<instance part="C4" gate="G$1" x="96.52" y="73.66" rot="R90"/>
-<instance part="C5" gate="G$1" x="106.68" y="60.96" rot="R180"/>
-<instance part="C6" gate="G$1" x="119.38" y="30.48" rot="R270"/>
-<instance part="+3V6" gate="G$1" x="129.54" y="30.48" rot="R270"/>
-<instance part="J2" gate="G$1" x="-7.62" y="55.88"/>
-<instance part="+3V7" gate="G$1" x="20.32" y="25.4" rot="R90"/>
 <instance part="U$4" gate="G$1" x="-5.08" y="25.4"/>
 <instance part="GND9" gate="1" x="-27.94" y="25.4" rot="R270"/>
-<instance part="C7" gate="G$1" x="48.26" y="5.08" rot="R270"/>
 <instance part="GND10" gate="1" x="48.26" y="40.64" rot="R270"/>
 <instance part="+3V3" gate="G$1" x="20.32" y="25.4" rot="R90"/>
@@
 <instance part="GND3" gate="1" x="53.34" y="-15.24" rot="R90"/>
 <instance part="R2" gate="G$1" x="5.08" y="-15.24"/>
-<instance part="+3V9" gate="G$1" x="-5.08" y="-15.24" rot="R90"/>
+<instance part="+3V9" gate="G$1" x="-7.62" y="-15.24" rot="R90"/>
 <instance part="J4" gate="G$1" x="71.12" y="-12.7"/>
 <instance part="J5" gate="G$1" x="116.84" y="0"/>
@@
 <pinref part="+3V2" gate="G$1" pin="+3V3"/>
 <wire x1="91.44" y1="50.8" x2="106.68" y2="50.8" width="0.1524" layer="91"/>
-<pinref part="C5" gate="G$1" pin="+"/>
-<wire x1="106.68" y1="58.42" x2="106.68" y2="50.8" width="0.1524" layer="91"/>
-<junction x="106.68" y="50.8"/>
 </segment>
 <segment>
@@
 <pinref part="+3V1" gate="G$1" pin="+3V3"/>
 <wire x1="91.44" y1="76.2" x2="104.14" y2="76.2" width="0.1524" layer="91"/>
-<wire x1="91.44" y1="76.2" x2="91.44" y2="73.66" width="0.1524" layer="91"/>
-<junction x="91.44" y="76.2"/>
-<pinref part="C4" gate="G$1" pin="+"/>
-<wire x1="91.44" y1="73.66" x2="93.98" y2="73.66" width="0.1524" layer="91"/>
 </segment>
 <segment>
@@
 </segment>
 <segment>
-<pinref part="+3V6" gate="G$1" pin="+3V3"/>
-<pinref part="C6" gate="G$1" pin="+"/>
-<wire x1="127" y1="30.48" x2="121.92" y2="30.48" width="0.1524" layer="91"/>
-</segment>
-<segment>
 <pinref part="R1" gate="G$1" pin="1"/>
-<pinref part="+3V7" gate="G$1" pin="+3V3"/>
 <wire x1="25.4" y1="25.4" x2="22.86" y2="25.4" width="0.1524" layer="91"/>
 <pinref part="+3V3" gate="G$1" pin="+3V3"/>
-<junction x="22.86" y="25.4"/>
 </segment>
 <segment>
 <pinref part="U$1" gate="G$1" pin="13.GND"/>
-<wire x1="38.1" y1="15.24" x2="40.64" y2="15.24" width="0.1524" layer="91"/>
-<wire x1="40.64" y1="15.24" x2="55.88" y2="15.24" width="0.1524" layer="91"/>
-<junction x="40.64" y="15.24"/>
-<wire x1="40.64" y1="15.24" x2="40.64" y2="5.08" width="0.1524" layer="91"/>
-<pinref part="C7" gate="G$1" pin="-"/>
-<wire x1="40.64" y1="5.08" x2="43.18" y2="5.08" width="0.1524" layer="91"/>
+<wire x1="38.1" y1="15.24" x2="55.88" y2="15.24" width="0.1524" layer="91"/>
 <pinref part="+3V8" gate="G$1" pin="+3V3"/>
 </segment>
@@
 </segment>
 <segment>
-<pinref part="+3V9" gate="G$1" pin="+3V3"/>
-<wire x1="-2.54" y1="-15.24" x2="2.54" y2="-15.24" width="0.1524" layer="91"/>
-</segment>
-<segment>
 <pinref part="J4" gate="G$1" pin="2"/>
 <wire x1="76.2" y1="-17.78" x2="78.74" y2="-17.78" width="0.1524" layer="91"/>
 <label x="78.74" y="-17.78" size="1.778" layer="95"/>
 </segment>
+<segment>
+<pinref part="+3V9" gate="G$1" pin="+3V3"/>
+<pinref part="R2" gate="G$1" pin="1"/>
+<wire x1="-5.08" y1="-15.24" x2="0" y2="-15.24" width="0.1524" layer="91"/>
+</segment>
 </net>
 <net name="GND" class="0">
@@
 <pinref part="GND1" gate="1" pin="GND"/>
 <wire x1="91.44" y1="71.12" x2="104.14" y2="71.12" width="0.1524" layer="91"/>
-<pinref part="C4" gate="G$1" pin="-"/>
-<wire x1="101.6" y1="73.66" x2="104.14" y2="71.12" width="0.1524" layer="91"/>
-<junction x="104.14" y="71.12"/>
-<pinref part="C5" gate="G$1" pin="-"/>
-<wire x1="106.68" y1="66.04" x2="106.68" y2="68.58" width="0.1524" layer="91"/>
-<wire x1="106.68" y1="68.58" x2="104.14" y2="68.58" width="0.1524" layer="91"/>
-<wire x1="104.14" y1="68.58" x2="104.14" y2="71.12" width="0.1524" layer="91"/>
 </segment>
 <segment>
@@
 <pinref part="GND2" gate="1" pin="GND"/>
 <wire x1="91.44" y1="30.48" x2="104.14" y2="30.48" width="0.1524" layer="91"/>
-<wire x1="104.14" y1="30.48" x2="104.14" y2="25.4" width="0.1524" layer="91"/>
-<junction x="104.14" y="30.48"/>
-<wire x1="104.14" y1="25.4" x2="111.76" y2="25.4" width="0.1524" layer="91"/>
-<wire x1="111.76" y1="25.4" x2="111.76" y2="30.48" width="0.1524" layer="91"/>
-<pinref part="C6" gate="G$1" pin="-"/>
-<wire x1="111.76" y1="30.48" x2="114.3" y2="30.48" width="0.1524" layer="91"/>
 </segment>
 <segment>
@@
 </segment>
 <segment>
-<pinref part="J1" gate="G$1" pin="GND"/>
 <pinref part="GND5" gate="1" pin="GND"/>
-<wire x1="129.54" y1="73.66" x2="127" y2="73.66" width="0.1524" layer="91"/>
-<wire x1="127" y1="73.66" x2="127" y2="63.5" width="0.1524" layer="91"/>
 <pinref part="C2" gate="G$1" pin="-"/>
 <wire x1="119.38" y1="66.04" x2="119.38" y2="63.5" width="0.1524" layer="91"/>
 <wire x1="119.38" y1="63.5" x2="127" y2="63.5" width="0.1524" layer="91"/>
-<junction x="127" y="63.5"/>
+<wire x1="127" y1="63.5" x2="127" y2="71.12" width="0.1524" layer="91"/>
+<pinref part="J1" gate="G$1" pin="1.GND"/>
+<wire x1="127" y1="71.12" x2="129.54" y2="71.12" width="0.1524" layer="91"/>
 </segment>
 <segment>
@@
 <wire x1="53.34" y1="40.64" x2="55.88" y2="40.64" width="0.1524" layer="91"/>
 <wire x1="53.34" y1="40.64" x2="53.34" y2="22.86" width="0.1524" layer="91"/>
-<pinref part="C7" gate="G$1" pin="+"/>
-<wire x1="53.34" y1="22.86" x2="53.34" y2="5.08" width="0.1524" layer="91"/>
-<wire x1="50.8" y1="5.08" x2="53.34" y2="5.08" width="0.1524" layer="91"/>
 <pinref part="GND10" gate="1" pin="GND"/>
 <wire x1="53.34" y1="40.64" x2="50.8" y2="40.64" width="0.1524" layer="91"/>
@@
 <wire x1="40.64" y1="20.32" x2="40.64" y2="22.86" width="0.1524" layer="91"/>
 <wire x1="40.64" y1="22.86" x2="53.34" y2="22.86" width="0.1524" layer="91"/>
-<junction x="53.34" y="22.86"/>
 </segment>
 <segment>
@@
 <wire x1="91.44" y1="45.72" x2="114.3" y2="45.72" width="0.1524" layer="91"/>
 <wire x1="114.3" y1="45.72" x2="114.3" y2="78.74" width="0.1524" layer="91"/>
-<pinref part="J1" gate="G$1" pin="D-"/>
-<wire x1="114.3" y1="78.74" x2="129.54" y2="78.74" width="0.1524" layer="91"/>
+<pinref part="J1" gate="G$1" pin="4.D-"/>
+<wire x1="129.54" y1="78.74" x2="114.3" y2="78.74" width="0.1524" layer="91"/>
 </segment>
 </net>
@@
 <segment>
 <pinref part="U$1" gate="G$1" pin="21.D+"/>
-<wire x1="91.44" y1="40.64" x2="144.78" y2="40.64" width="0.1524" layer="91"/>
-<wire x1="144.78" y1="40.64" x2="144.78" y2="86.36" width="0.1524" layer="91"/>
-<wire x1="144.78" y1="86.36" x2="124.46" y2="86.36" width="0.1524" layer="91"/>
-<wire x1="124.46" y1="86.36" x2="124.46" y2="81.28" width="0.1524" layer="91"/>
-<pinref part="J1" gate="G$1" pin="D+"/>
-<wire x1="124.46" y1="81.28" x2="129.54" y2="81.28" width="0.1524" layer="91"/>
+<wire x1="91.44" y1="40.64" x2="147.32" y2="40.64" width="0.1524" layer="91"/>
+<wire x1="147.32" y1="40.64" x2="147.32" y2="76.2" width="0.1524" layer="91"/>
+<pinref part="J1" gate="G$1" pin="3.D+"/>
+<wire x1="147.32" y1="76.2" x2="129.54" y2="76.2" width="0.1524" layer="91"/>
 </segment>
 </net>
@@
 <wire x1="55.88" y1="10.16" x2="43.18" y2="10.16" width="0.1524" layer="91"/>
 <label x="43.18" y="10.16" size="1.778" layer="95"/>
+</segment>
+<segment>
+<pinref part="J1" gate="G$1" pin="2.ID"/>
+<wire x1="129.54" y1="73.66" x2="124.46" y2="73.66" width="0.1524" layer="91"/>
+<wire x1="124.46" y1="73.66" x2="124.46" y2="58.42" width="0.1524" layer="91"/>
+<label x="124.46" y="58.42" size="1.778" layer="95"/>
 </segment>
 </net>
@@
 <net name="N$6" class="0">
 <segment>
-<pinref part="J1" gate="G$1" pin="VBUS"/>
-<wire x1="129.54" y1="76.2" x2="121.92" y2="76.2" width="0.1524" layer="91"/>
 <wire x1="121.92" y1="76.2" x2="121.92" y2="88.9" width="0.1524" layer="91"/>
 <wire x1="121.92" y1="88.9" x2="104.14" y2="88.9" width="0.1524" layer="91"/>
 <pinref part="U$5" gate="G$1" pin="1.5V"/>
 <wire x1="104.14" y1="88.9" x2="104.14" y2="91.44" width="0.1524" layer="91"/>
-</segment>
-</net>
+<wire x1="121.92" y1="76.2" x2="127" y2="76.2" width="0.1524" layer="91"/>
+<wire x1="127" y1="76.2" x2="127" y2="81.28" width="0.1524" layer="91"/>
+<pinref part="J1" gate="G$1" pin="5.VBUS"/>
+<wire x1="127" y1="81.28" x2="129.54" y2="81.28" width="0.1524" layer="91"/>
+</segment>
+</net>

Commit message: gerber files complete! PCB ready for printing
Parts:
- removed J1: USBSMD, pic32_library:USBSMD
- added J2: USB-MB-H, pic32_library:USB-MB-H
- renumbered U$1 to PIC32
Connections:
- net GND: now also J2.1.GND; no longer J1.1.GND
- net N$2: now also J2.4.D-; no longer J1.4.D-
- net N$3: now also J2.3.D+; no longer J1.3.D+
- net N$6: now also J2.5.VBUS; no longer J1.5.VBUS
- net USBID: now also J2.2.ID; no longer J1.2.ID
